Commit message: added unite_imu_method

File: urdf/_d435i.gazebo.xacro (robot description, xacro)
@@ -9,5 +9,5 @@
 -->
 <robot xmlns:xacro="http://ros.org/wiki/xacro">
-  <xacro:macro name="gazebo_d435i" params="camera_name reference_link topics_ns depth_optical_frame color_optical_frame infrared1_optical_frame infrared2_optical_frame accel_optical_frame gyro_optical_frame enable_pointCloud:=false">
+  <xacro:macro name="gazebo_d435i" params="camera_name reference_link topics_ns depth_optical_frame color_optical_frame infrared1_optical_frame infrared2_optical_frame accel_optical_frame gyro_optical_frame enable_pointCloud:=false unite_imu_method:=false">
     <!-- Load parameters to model's main link-->
     <xacro:property name="deg_to_rad" value="0.01745329251994329577"/>
@@ -114,36 +114,55 @@
         <visualize>0</visualize>
       </sensor>
-      <sensor name="{camera_name}accel" type="imu">
-        <always_on>true</always_on>
-        <update_rate>300</update_rate>
-        <topic>${camera_name}/accel/sample</topic>
-        <plugin name="${topics_ns}_accel_plugin" filename="librealsense_gazebo_accel_sensor.so">
-          <topicName>${camera_name}/accel/sample</topicName>
-          <bodyName>imu_link</bodyName>
-          <updateRateHZ>300.0</updateRateHZ>
-          <gaussianNoise>0.1</gaussianNoise>
-          <xyzOffset>0 0 0</xyzOffset>
-          <rpyOffset>0 0 0</rpyOffset>
-          <frameName>${accel_optical_frame}</frameName>
-          <initialOrientationAsReference>false</initialOrientationAsReference>
-        </plugin>
-        <pose>0 0 0 0 0 0</pose>
-      </sensor>
-      <sensor name="{camera_name}gyro" type="imu">
-        <always_on>true</always_on>
-        <update_rate>300</update_rate>
-        <topic>${camera_name}/gyro/sample</topic>
-        <plugin name="${topics_ns}_gyro_plugin" filename="librealsense_gazebo_gyro_sensor.so">
-          <topicName>${camera_name}/gyro/sample</topicName>
-          <bodyName>imu_link</bodyName>
-          <updateRateHZ>300.0</updateRateHZ>
-          <gaussianNoise>0.1</gaussianNoise>
-          <xyzOffset>0 0 0</xyzOffset>
-          <rpyOffset>0 0 0</rpyOffset>
-          <frameName>${gyro_optical_frame}</frameName>
-          <initialOrientationAsReference>false</initialOrientationAsReference>
-        </plugin>
-        <pose>0 0 0 0 0 0</pose>
-      </sensor>
+      <!-- IMU -->
+      <xacro:if value="${unite_imu_method == 'copy' or unite_imu_method == 'linear_interpolation'}">
+        <sensor name="${camera_name}_imu" type="imu">
+          <always_on>true</always_on>
+          <update_rate>300</update_rate>
+          <topic>${camera_name}/imu/sample</topic>
+          <plugin name="{camera_name}imu" filename="libgazebo_ros_imu_sensor.so">
+            <topicName>${camera_name}/imu/sample</topicName>
+            <bodyName>${camera_name}_link</bodyName>
+            <frameName>${gyro_optical_frame}</frameName>
+            <updateRateHZ>300</updateRateHZ>
+            <gaussianNoise>0.1</gaussianNoise>
+            <xyzOffset>0 0 0</xyzOffset>
+            <rpyOffset>0 0 0</rpyOffset>
+          </plugin>
+        </sensor>
+      </xacro:if>
+      <!-- Accel and gyro -->
+      <xacro:unless value="${unite_imu_method == 'copy' or unite_imu_method == 'linear_interpolation'}">
+        <sensor name="{camera_name}accel" type="imu">
+          <always_on>true</always_on>
+          <update_rate>300</update_rate>
+          <topic>${camera_name}/accel/sample</topic>
+          <plugin name="${topics_ns}_accel_plugin" filename="librealsense_gazebo_accel_sensor.so">
+            <topicName>${camera_name}/accel/sample</topicName>
+            <bodyName>${camera_name}_link</bodyName>
+            <updateRateHZ>300.0</updateRateHZ>
+            <gaussianNoise>0.1</gaussianNoise>
+            <xyzOffset>0 0 0</xyzOffset>
+            <rpyOffset>0 0 0</rpyOffset>
+            <frameName>${accel_optical_frame}</frameName>
+            <initialOrientationAsReference>false</initialOrientationAsReference>
+          </plugin>
+          <pose>0 0 0 0 0 0</pose>
+        </sensor>
+        <sensor name="{camera_name}gyro" type="imu">
+          <always_on>true</always_on>
+          <update_rate>300</update_rate>
+          <topic>${camera_name}/gyro/sample</topic>
+          <plugin name="${topics_ns}_gyro_plugin" filename="librealsense_gazebo_gyro_sensor.so">
+            <topicName>${camera_name}/gyro/sample</topicName>
+            <bodyName>${camera_name}_link</bodyName>
+            <updateRateHZ>300.0</updateRateHZ>
+            <gaussianNoise>0.1</gaussianNoise>
+            <xyzOffset>0 0 0</xyzOffset>
+            <rpyOffset>0 0 0</rpyOffset>
+            <frameName>${gyro_optical_frame}</frameName>
+            <initialOrientationAsReference>false</initialOrientationAsReference>
+          </plugin>
+        </sensor>
+      </xacro:unless>
     </gazebo>
     <gazebo>

File: urdf/_d435i.urdf.xacro (robot description, xacro)
@@ -12,5 +12,5 @@
   <!--File includes-->
   <xacro:include filename="$(find realsense_gazebo_description)/urdf/_d435i.gazebo.xacro"/>
-  <xacro:macro name="sensor_d435i" params="name:=camera topics_ns:=camera parent enable_pointCloud:=false align_depth=false *origin">
+  <xacro:macro name="sensor_d435i" params="name:=camera topics_ns:=camera parent enable_pointCloud:=false align_depth=false unite_imu_method:=false *origin">
     <xacro:property name="M_PI" value="3.1415926535897931"/>
     <!-- The following values are approximate, and the camera node
@@ -158,4 +158,5 @@
                         gyro_optical_frame="${name}_gyro_optical_frame"
                         enable_pointCloud="${enable_pointCloud}"
+                        unite_imu_method="${unite_imu_method}"
     />
     <xacro:if value="${align_depth}">

File: urdf/_t265.gazebo.xacro (robot description, xacro)
@@ -9,5 +9,5 @@
 -->
 <robot xmlns:xacro="http://ros.org/wiki/xacro">
-  <xacro:macro name="gazebo_t265" params="camera_name fisheye1_reference_link fisheye2_reference_link topics_ns fisheye1_optical_frame fisheye2_optical_frame accel_optical_frame gyro_optical_frame pose_frame xyz rpy odom_rate:=200" >
+  <xacro:macro name="gazebo_t265" params="camera_name fisheye1_reference_link fisheye2_reference_link topics_ns fisheye1_optical_frame fisheye2_optical_frame accel_optical_frame gyro_optical_frame pose_frame xyz rpy odom_rate:=200 unite_imu_method:=false">
     <!-- Load parameters to model's main link-->
     <gazebo reference="${fisheye1_reference_link}">
@@ -126,35 +126,54 @@
         </plugin>
       </sensor>
+      <!-- IMU -->
+      <xacro:if value="${unite_imu_method == 'copy' or unite_imu_method == 'linear_interpolation'}">
+        <sensor name="${camera_name}_imu" type="imu">
+          <always_on>true</always_on>
+          <update_rate>300</update_rate>
+          <topic>${camera_name}/imu/sample</topic>
+          <plugin name="{camera_name}imu" filename="libgazebo_ros_imu_sensor.so">
+            <topicName>${camera_name}/imu/sample</topicName>
+            <bodyName>${camera_name}_pose_frame</bodyName>
+            <frameName>${gyro_optical_frame}</frameName>
+            <updateRateHZ>300</updateRateHZ>
+            <gaussianNoise>0.1</gaussianNoise>
+            <xyzOffset>0 0 0</xyzOffset>
+            <rpyOffset>0 0 0</rpyOffset>
+          </plugin>
+        </sensor>
+      </xacro:if>
       <!-- Accel and gyro -->
-      <sensor name="{camera_name}accel" type="imu">
-        <always_on>true</always_on>
-        <update_rate>300</update_rate>
-        <topic>${topics_ns}/accel/sample</topic>
-        <plugin name="${topics_ns}_accel_plugin" filename="librealsense_gazebo_accel_sensor.so">
-          <topicName>${camera_name}/accel/sample</topicName>
-          <bodyName>imu_accel_link</bodyName>
-          <updateRateHZ>300.0</updateRateHZ>
-          <gaussianNoise>0.1</gaussianNoise>
-          <xyzOffset>0 0 0</xyzOffset>
-          <rpyOffset>0 0 0</rpyOffset>
-          <frameName>${accel_optical_frame}</frameName>
-        </plugin>
-        <pose>0 0 0 0 0 0</pose>
-      </sensor>
-      <sensor name="{camera_name}gyro" type="imu">
-        <pose>0 0 0 0 0 0</pose>
-        <always_on>true</always_on>
-        <update_rate>300</update_rate>
-        <topic>${topics_ns}/gyro/sample</topic>
-        <plugin name="${topics_ns}_gyro_plugin" filename="librealsense_gazebo_gyro_sensor.so">
-          <topicName>${camera_name}/gyro/sample</topicName>
-          <bodyName>imu_gyro_link</bodyName>
-          <updateRateHZ>300.0</updateRateHZ>
-          <gaussianNoise>0.1</gaussianNoise>
-          <xyzOffset>0 0 0</xyzOffset>
-          <rpyOffset>0 0 0</rpyOffset>
-          <frameName>${gyro_optical_frame}</frameName>
-        </plugin>
-      </sensor>
+      <xacro:unless value="${unite_imu_method == 'copy' or unite_imu_method == 'linear_interpolation'}">
+        <sensor name="{camera_name}accel" type="imu">
+          <always_on>true</always_on>
+          <update_rate>300</update_rate>
+          <plugin name="${topics_ns}_accel_plugin" filename="librealsense_gazebo_accel_sensor.so">
+            <topicName>${camera_name}/accel/sample</topicName>
+            <bodyName>${camera_name}_pose_frame</bodyName>
+            <updateRateHZ>300.0</updateRateHZ>
+            <gaussianNoise>0.1</gaussianNoise>
+            <xyzOffset>0 0 0</xyzOffset>
+            <rpyOffset>0 0 0</rpyOffset>
+            <frameName>${accel_optical_frame}</frameName>
+            <initialOrientationAsReference>false</initialOrientationAsReference>
+          </plugin>
+          <pose>0 0 0 0 0 0</pose>
+        </sensor>
+        <sensor name="{camera_name}gyro" type="imu">
+          <always_on>true</always_on>
+          <update_rate>300</update_rate>
+          <topic>${topics_ns}/gyro/sample</topic>
+          <plugin name="${topics_ns}_gyro_plugin" filename="librealsense_gazebo_gyro_sensor.so">
+            <topicName>${camera_name}/gyro/sample</topicName>
+            <bodyName>${camera_name}_pose_frame</bodyName>
+            <updateRateHZ>300.0</updateRateHZ>
+            <gaussianNoise>0.1</gaussianNoise>
+            <xyzOffset>0 0 0</xyzOffset>
+            <rpyOffset>0 0 0</rpyOffset>
+            <frameName>${gyro_optical_frame}</frameName>
+            <initialOrientationAsReference>false</initialOrientationAsReference>
+          </plugin>
+        </sensor>
+      </xacro:unless>
     </gazebo>
     <gazebo>

File: urdf/_t265.urdf.xacro (robot description, xacro)
@@ -14,5 +14,5 @@
   <!-- tx,ty,tz,rr,rp,ry (xyz rpy) are the transformation from the robot base_link to the camera reference frame (camerea_pose_frame)
   they are needed for the simulation of the camera slam capabilities -->
-  <xacro:macro name="sensor_t265" params="parent xyz rpy name:=camera topics_ns:=camera odom_rate:=200 *origin">
+  <xacro:macro name="sensor_t265" params="parent xyz rpy name:=camera topics_ns:=camera odom_rate:=200 unite_imu_method:=false *origin">
     <xacro:property name="M_PI" value="3.1415926535897931"/>
     <!-- The following values are approximate, and the camera node
@@ -123,4 +123,5 @@
                         xyz="${xyz}"
                         rpy="${rpy}"
+                        unite_imu_method="${unite_imu_method}"
     />
     <!--

File: urdf/multicamera.urdf.xacro (robot description, xacro)
@@ -11,5 +11,6 @@
   <xacro:include filename="$(find realsense_gazebo_description)/urdf/_d435i.urdf.xacro"/>
   <xacro:sensor_d435i parent="base_link" name="D435i_camera" topics_ns="D435i_camera"
-                      enable_pointCloud="true" align_depth="true">
+                      enable_pointCloud="true" align_depth="true"
+                      unite_imu_method="copy"> <!-- unite_imu_method can be false, copy or linear_interpolation -->
     <origin xyz="0.0 0.5 0.1" rpy="0.0 0.0 0.0"/>
   </xacro:sensor_d435i>
@@ -17,5 +18,6 @@
   <xacro:include filename="$(find realsense_gazebo_description)/urdf/_t265.urdf.xacro"/>
   <xacro:sensor_t265  parent="base_link" name="T265_camera" topics_ns="T265_camera"
-                      xyz="0.0 0.0 0.25" rpy="0.0 0.0 0.0">
+                      xyz="0.0 0.0 0.25" rpy="0.0 0.0 0.0"
+                      unite_imu_method="false"> <!-- unite_imu_method can be false, copy or linear_interpolation -->
     <origin xyz="0.0 0.0 0.25" rpy="0.0 0.0 0.0"/>
   </xacro:sensor_t265>

Commit message: added unite_imu_method

File: urdf/_d435i.gazebo.xacro (robot description, xacro)
@@ -9,5 +9,5 @@
 -->
 <robot xmlns:xacro="http://ros.org/wiki/xacro">
-  <xacro:macro name="gazebo_d435i" params="camera_name reference_link topics_ns depth_optical_frame color_optical_frame infrared1_optical_frame infrared2_optical_frame accel_optical_frame gyro_optical_frame" >
+  <xacro:macro name="gazebo_d435i" params="camera_name reference_link topics_ns depth_optical_frame color_optical_frame infrared1_optical_frame infrared2_optical_frame accel_optical_frame gyro_optical_frame enable_pointCloud:=false unite_imu_method:=false">
     <!-- Load parameters to model's main link-->
     <xacro:property name="deg_to_rad" value="0.01745329251994329577"/>
@@ -113,34 +113,55 @@
         <visualize>0</visualize>
       </sensor>
-      <sensor name="{camera_name}accel" type="imu">
-        <always_on>true</always_on>
-        <update_rate>300</update_rate>
-        <topic>${camera_name}/accel/sample</topic>
-        <plugin name="${topics_ns}_accel_plugin" filename="librealsense_gazebo_accel_sensor.so">
-          <topicName>${camera_name}/accel/sample</topicName>
-          <bodyName>imu_link</bodyName>
-          <updateRateHZ>300.0</updateRateHZ>
-          <gaussianNoise>0.1</gaussianNoise>
-          <xyzOffset>0 0 0</xyzOffset>
-          <rpyOffset>0 0 0</rpyOffset>
-          <frameName>${accel_optical_frame}</frameName>
-        </plugin>
-        <pose>0 0 0 0 0 0</pose>
-      </sensor>
-      <sensor name="{camera_name}gyro" type="imu">
-        <always_on>true</always_on>
-        <update_rate>300</update_rate>
-        <topic>${camera_name}/gyro/sample</topic>
-        <plugin name="${topics_ns}_gyro_plugin" filename="librealsense_gazebo_gyro_sensor.so">
-          <topicName>${camera_name}/gyro/sample</topicName>
-          <bodyName>imu_link</bodyName>
-          <updateRateHZ>300.0</updateRateHZ>
-          <gaussianNoise>0.1</gaussianNoise>
-          <xyzOffset>0 0 0</xyzOffset>
-          <rpyOffset>0 0 0</rpyOffset>
-          <frameName>${gyro_optical_frame}</frameName>
-        </plugin>
-        <pose>0 0 0 0 0 0</pose>
-      </sensor>
+      <!-- IMU -->
+      <xacro:if value="${unite_imu_method == 'copy' or unite_imu_method == 'linear_interpolation'}">
+        <sensor name="${camera_name}_imu" type="imu">
+          <always_on>true</always_on>
+          <update_rate>300</update_rate>
+          <topic>${camera_name}/imu/sample</topic>
+          <plugin name="{camera_name}imu" filename="libgazebo_ros_imu_sensor.so">
+            <topicName>${camera_name}/imu/sample</topicName>
+            <bodyName>${camera_name}_link</bodyName>
+            <frameName>${gyro_optical_frame}</frameName>
+            <updateRateHZ>300</updateRateHZ>
+            <gaussianNoise>0.1</gaussianNoise>
+            <xyzOffset>0 0 0</xyzOffset>
+            <rpyOffset>0 0 0</rpyOffset>
+          </plugin>
+        </sensor>
+      </xacro:if>
+      <!-- Accel and gyro -->
+      <xacro:unless value="${unite_imu_method == 'copy' or unite_imu_method == 'linear_interpolation'}">
+        <sensor name="{camera_name}accel" type="imu">
+          <always_on>true</always_on>
+          <update_rate>300</update_rate>
+          <topic>${camera_name}/accel/sample</topic>
+          <plugin name="${topics_ns}_accel_plugin" filename="librealsense_gazebo_accel_sensor.so">
+            <topicName>${camera_name}/accel/sample</topicName>
+            <bodyName>${camera_name}_link</bodyName>
+            <updateRateHZ>300.0</updateRateHZ>
+            <gaussianNoise>0.1</gaussianNoise>
+            <xyzOffset>0 0 0</xyzOffset>
+            <rpyOffset>0 0 0</rpyOffset>
+            <frameName>${accel_optical_frame}</frameName>
+            <initialOrientationAsReference>false</initialOrientationAsReference>
+          </plugin>
+          <pose>0 0 0 0 0 0</pose>
+        </sensor>
+        <sensor name="{camera_name}gyro" type="imu">
+          <always_on>true</always_on>
+          <update_rate>300</update_rate>
+          <topic>${camera_name}/gyro/sample</topic>
+          <plugin name="${topics_ns}_gyro_plugin" filename="librealsense_gazebo_gyro_sensor.so">
+            <topicName>${camera_name}/gyro/sample</topicName>
+            <bodyName>${camera_name}_link</bodyName>
+            <updateRateHZ>300.0</updateRateHZ>
+            <gaussianNoise>0.1</gaussianNoise>
+            <xyzOffset>0 0 0</xyzOffset>
+            <rpyOffset>0 0 0</rpyOffset>
+            <frameName>${gyro_optical_frame}</frameName>
+            <initialOrientationAsReference>false</initialOrientationAsReference>
+          </plugin>
+        </sensor>
+      </xacro:unless>
     </gazebo>
     <gazebo>
@@ -164,5 +185,5 @@
       	<rangeMinDepth>0.2</rangeMinDepth>
       	<rangeMaxDepth>10.0</rangeMaxDepth>
-      	<pointCloud>true</pointCloud>
+      	<pointCloud>${enable_pointCloud}</pointCloud>
       	<pointCloudTopicName>depth/points</pointCloudTopicName>
       	<pointCloudCutoff>0.5</pointCloudCutoff>

File: urdf/_d435i.urdf.xacro (robot description, xacro)
@@ -12,5 +12,5 @@
   <!--File includes-->
   <xacro:include filename="$(find realsense_gazebo_description)/urdf/_d435i.gazebo.xacro"/>
-  <xacro:macro name="sensor_d435i" params="name:=camera topics_ns:=camera parent *origin">
+  <xacro:macro name="sensor_d435i" params="name:=camera topics_ns:=camera parent enable_pointCloud:=false unite_imu_method:=false *origin">
     <xacro:property name="M_PI" value="3.1415926535897931"/>
     <!-- The following values are approximate, and the camera node
@@ -157,4 +157,6 @@
                         accel_optical_frame="${name}_accel_optical_frame"
                         gyro_optical_frame="${name}_gyro_optical_frame"
+                        enable_pointCloud="${enable_pointCloud}"
+                        unite_imu_method="${unite_imu_method}"
     />
   </xacro:macro>

File: urdf/multicamera.urdf.xacro (robot description, xacro)
@@ -9,11 +9,13 @@
   <!-- d435i frame definition can be found at https://github.com/IntelRealSense/librealsense/blob/master/doc/d435i.md -->
   <xacro:include filename="$(find realsense_gazebo_description)/urdf/_d435i.urdf.xacro"/>
-  <xacro:sensor_d435i parent="base_link" name="D435i_camera" topics_ns="D435i_camera">
+  <xacro:sensor_d435i parent="base_link" name="D435i_camera" topics_ns="D435i_camera"
+                      enable_pointCloud="true" unite_imu_method="copy"> <!-- unite_imu_method can be false, copy or linear_interpolation -->
     <origin xyz="0.0 0.5 0.1" rpy="0.0 0.0 0.0"/>
   </xacro:sensor_d435i>
   <!-- t265  frame definition can be found at https://github.com/IntelRealSense/librealsense/blob/master/doc/t265.md -->
   <xacro:include filename="$(find realsense_gazebo_description)/urdf/_t265.urdf.xacro"/>
-  <xacro:sensor_t265  parent="base_link" name="CL_camera" topics_ns="CL_camera"
-                      xyz="0.0 0.0 0.0" rpy="0.0 0.0 0.0">
+  <xacro:sensor_t265  parent="base_link" name="T265_camera" topics_ns="T265_camera"
+                      xyz="0.0 0.0 0.25" rpy="0.0 0.0 0.0"
+                      unite_imu_method="false"> <!-- unite_imu_method can be false, copy or linear_interpolation -->
     <origin xyz="0.0 0.0 0.25" rpy="0.0 0.0 0.0"/>
   </xacro:sensor_t265>
