Commit message: added aligned_depth_to_color for d435 and d435i

File: urdf/_d435.gazebo.xacro (robot description, xacro)
@@ -8,5 +8,5 @@
 -->
 <robot xmlns:xacro="http://ros.org/wiki/xacro">
-  <xacro:macro name="gazebo_d435" params="camera_name reference_link topics_ns depth_optical_frame color_optical_frame infrared1_optical_frame infrared2_optical_frame" >
+  <xacro:macro name="gazebo_d435" params="camera_name reference_link topics_ns depth_optical_frame color_optical_frame infrared1_optical_frame infrared2_optical_frame enable_pointCloud:=false">
     <!-- Load parameters to model's main link-->
     <xacro:property name="deg_to_rad" value="0.01745329251994329577"/>
@@ -119,11 +119,11 @@
       	<colorUpdateRate>60.0</colorUpdateRate>
       	<infraredUpdateRate>60.0</infraredUpdateRate>
-      	<depthTopicName>depth/image_raw</depthTopicName>
+      	<depthTopicName>depth/image_rect_raw</depthTopicName>
       	<depthCameraInfoTopicName>depth/camera_info</depthCameraInfoTopicName>
       	<colorTopicName>color/image_raw</colorTopicName>
       	<colorCameraInfoTopicName>color/camera_info</colorCameraInfoTopicName>
-      	<infrared1TopicName>infra1/image_raw</infrared1TopicName>
+      	<infrared1TopicName>infra1/image_rect_raw</infrared1TopicName>
       	<infrared1CameraInfoTopicName>infra1/camera_info</infrared1CameraInfoTopicName>
-      	<infrared2TopicName>infra2/image_raw</infrared2TopicName>
+      	<infrared2TopicName>infra2/image_rect_raw</infrared2TopicName>
       	<infrared2CameraInfoTopicName>infra2/camera_info</infrared2CameraInfoTopicName>
       	<colorOpticalframeName>${color_optical_frame}</colorOpticalframeName>
@@ -133,6 +133,6 @@
       	<rangeMinDepth>0.2</rangeMinDepth>
       	<rangeMaxDepth>10.0</rangeMaxDepth>
-      	<pointCloud>true</pointCloud>
-      	<pointCloudTopicName>depth/points</pointCloudTopicName>
+      	<pointCloud>${enable_pointCloud}</pointCloud>
+      	<pointCloudTopicName>depth/color/points</pointCloudTopicName>
       	<pointCloudCutoff>0.5</pointCloudCutoff>
       </plugin>

File: urdf/_d435.urdf.xacro (robot description, xacro)
@@ -12,5 +12,5 @@
   <!--File includes-->
   <xacro:include filename="$(find realsense_gazebo_description)/urdf/_d435.gazebo.xacro"/>
-  <xacro:macro name="sensor_d435" params="name:=camera topics_ns:=camera parent *origin">
+  <xacro:macro name="sensor_d435" params="name:=camera topics_ns:=camera parent enable_pointCloud:=false align_depth=false *origin">
     <xacro:property name="M_PI" value="3.1415926535897931"/>
     <!-- The following values are approximate, and the camera node
@@ -123,11 +123,21 @@
     <!-- Realsense Gazebo Plugin -->
     <xacro:gazebo_d435  camera_name="${name}"
+                        topics_ns="${topics_ns}"
                         reference_link="${name}_link"
-                        topics_ns="${topics_ns}"
                         depth_optical_frame="${name}_depth_optical_frame"
                         color_optical_frame="${name}_color_optical_frame"
                         infrared1_optical_frame="${name}_left_ir_optical_frame"
                         infrared2_optical_frame="${name}_right_ir_optical_frame"
+                        enable_pointCloud="${enable_pointCloud}"
     />
+    <xacro:if value="${align_depth}">
+      <xacro:include filename="$(find realsense_gazebo_description)/urdf/realsense_align_depth.gazebo.xacro"/>
+      <xacro:gazebo_realsense_aligned_depth
+                          camera_name="${name}"
+                          topics_ns="${topics_ns}"
+                          reference_link="${name}_link"
+                          depth_optical_frame="${name}_depth_optical_frame"
+      />
+    </xacro:if>
   </xacro:macro>
 </robot>

File: urdf/_d435i.gazebo.xacro (robot description, xacro)
@@ -9,5 +9,5 @@
 -->
 <robot xmlns:xacro="http://ros.org/wiki/xacro">
-  <xacro:macro name="gazebo_d435i" params="camera_name reference_link topics_ns depth_optical_frame color_optical_frame infrared1_optical_frame infrared2_optical_frame accel_optical_frame gyro_optical_frame" >
+  <xacro:macro name="gazebo_d435i" params="camera_name reference_link topics_ns depth_optical_frame color_optical_frame infrared1_optical_frame infrared2_optical_frame accel_optical_frame gyro_optical_frame enable_pointCloud:=false">
     <!-- Load parameters to model's main link-->
     <xacro:property name="deg_to_rad" value="0.01745329251994329577"/>
@@ -96,4 +96,5 @@
           <horizontal_fov>${85.2*deg_to_rad}</horizontal_fov>
           <image>
+            <format>RGB_INT8</format>
             <width>1280</width>
             <height>720</height>
@@ -125,4 +126,5 @@
           <rpyOffset>0 0 0</rpyOffset>
           <frameName>${accel_optical_frame}</frameName>
+          <initialOrientationAsReference>false</initialOrientationAsReference>
         </plugin>
         <pose>0 0 0 0 0 0</pose>
@@ -140,4 +142,5 @@
           <rpyOffset>0 0 0</rpyOffset>
           <frameName>${gyro_optical_frame}</frameName>
+          <initialOrientationAsReference>false</initialOrientationAsReference>
         </plugin>
         <pose>0 0 0 0 0 0</pose>
@@ -150,11 +153,11 @@
       	<colorUpdateRate>60.0</colorUpdateRate>
       	<infraredUpdateRate>60.0</infraredUpdateRate>
-      	<depthTopicName>depth/image_raw</depthTopicName>
+      	<depthTopicName>depth/image_rect_raw</depthTopicName>
       	<depthCameraInfoTopicName>depth/camera_info</depthCameraInfoTopicName>
       	<colorTopicName>color/image_raw</colorTopicName>
       	<colorCameraInfoTopicName>color/camera_info</colorCameraInfoTopicName>
-      	<infrared1TopicName>infra1/image_raw</infrared1TopicName>
+      	<infrared1TopicName>infra1/image_rect_raw</infrared1TopicName>
       	<infrared1CameraInfoTopicName>infra1/camera_info</infrared1CameraInfoTopicName>
-      	<infrared2TopicName>infra2/image_raw</infrared2TopicName>
+      	<infrared2TopicName>infra2/image_rect_raw</infrared2TopicName>
       	<infrared2CameraInfoTopicName>infra2/camera_info</infrared2CameraInfoTopicName>
       	<colorOpticalframeName>${color_optical_frame}</colorOpticalframeName>
@@ -164,6 +167,6 @@
       	<rangeMinDepth>0.2</rangeMinDepth>
       	<rangeMaxDepth>10.0</rangeMaxDepth>
-      	<pointCloud>true</pointCloud>
-      	<pointCloudTopicName>depth/points</pointCloudTopicName>
+      	<pointCloud>${enable_pointCloud}</pointCloud>
+      	<pointCloudTopicName>depth/color/points</pointCloudTopicName>
       	<pointCloudCutoff>0.5</pointCloudCutoff>
       </plugin>

File: urdf/_d435i.urdf.xacro (robot description, xacro)
@@ -12,5 +12,5 @@
   <!--File includes-->
   <xacro:include filename="$(find realsense_gazebo_description)/urdf/_d435i.gazebo.xacro"/>
-  <xacro:macro name="sensor_d435i" params="name:=camera topics_ns:=camera parent *origin">
+  <xacro:macro name="sensor_d435i" params="name:=camera topics_ns:=camera parent enable_pointCloud:=false align_depth=false *origin">
     <xacro:property name="M_PI" value="3.1415926535897931"/>
     <!-- The following values are approximate, and the camera node
@@ -157,5 +157,15 @@
                         accel_optical_frame="${name}_accel_optical_frame"
                         gyro_optical_frame="${name}_gyro_optical_frame"
+                        enable_pointCloud="${enable_pointCloud}"
     />
+    <xacro:if value="${align_depth}">
+      <xacro:include filename="$(find realsense_gazebo_description)/urdf/realsense_align_depth.gazebo.xacro"/>
+      <xacro:gazebo_realsense_aligned_depth
+                          camera_name="${name}"
+                          topics_ns="${topics_ns}"
+                          reference_link="${name}_link"
+                          depth_optical_frame="${name}_depth_optical_frame"
+      />
+    </xacro:if>
   </xacro:macro>
 </robot>

File: urdf/multicamera.urdf.xacro (robot description, xacro)
@@ -4,16 +4,18 @@
   <!-- d435  frame definition can be found at https://github.com/IntelRealSense/librealsense/blob/master/doc/d435i.md -->
   <xacro:include filename="$(find realsense_gazebo_description)/urdf/_d435.urdf.xacro"/>
-  <xacro:sensor_d435 parent="base_link" name="D435_camera" topics_ns="D435_camera">
+  <xacro:sensor_d435  parent="base_link" name="D435_camera" topics_ns="D435_camera"
+                      enable_pointCloud="true" align_depth="true">
     <origin xyz="0.0 -0.5 0.1" rpy="0.0 0.0 0.0"/>
   </xacro:sensor_d435>
   <!-- d435i frame definition can be found at https://github.com/IntelRealSense/librealsense/blob/master/doc/d435i.md -->
   <xacro:include filename="$(find realsense_gazebo_description)/urdf/_d435i.urdf.xacro"/>
-  <xacro:sensor_d435i parent="base_link" name="D435i_camera" topics_ns="D435i_camera">
+  <xacro:sensor_d435i parent="base_link" name="D435i_camera" topics_ns="D435i_camera"
+                      enable_pointCloud="true" align_depth="true">
     <origin xyz="0.0 0.5 0.1" rpy="0.0 0.0 0.0"/>
   </xacro:sensor_d435i>
   <!-- t265  frame definition can be found at https://github.com/IntelRealSense/librealsense/blob/master/doc/t265.md -->
   <xacro:include filename="$(find realsense_gazebo_description)/urdf/_t265.urdf.xacro"/>
-  <xacro:sensor_t265  parent="base_link" name="CL_camera" topics_ns="CL_camera"
-                      xyz="0.0 0.0 0.0" rpy="0.0 0.0 0.0">
+  <xacro:sensor_t265  parent="base_link" name="T265_camera" topics_ns="T265_camera"
+                      xyz="0.0 0.0 0.25" rpy="0.0 0.0 0.0">
     <origin xyz="0.0 0.0 0.25" rpy="0.0 0.0 0.0"/>
   </xacro:sensor_t265>

Commit message: [bugfix] removed <gravity> and Element[origin] warnings

File: urdf/_d435.gazebo.xacro (robot description, xacro)
@@ -15,5 +15,5 @@
       <enable_wind>0</enable_wind>
       <kinematic>0</kinematic>
-      <gravity>1</gravity>
+      <!-- <gravity>1</gravity> -->
       <!--<mu>1</mu>-->
       <mu2>1</mu2>

File: urdf/_d435i.gazebo.xacro (robot description, xacro)
@@ -16,5 +16,5 @@
       <enable_wind>0</enable_wind>
       <kinematic>0</kinematic>
-      <gravity>1</gravity>
+      <!-- <gravity>1</gravity> -->
       <!--<mu>1</mu>-->
       <mu2>1</mu2>

File: urdf/_t265.gazebo.xacro (robot description, xacro)
@@ -15,5 +15,5 @@
       <enable_wind>0</enable_wind>
       <kinematic>0</kinematic>
-      <gravity>1</gravity>
+      <!-- <gravity>1</gravity> -->
       <!--<mu>1</mu>-->
       <mu2>1</mu2>
@@ -26,5 +26,5 @@
       <min_depth>0</min_depth>-->
       <sensor name="${camera_name}fisheye1" type="wideanglecamera">
-        <origin xyz="0 0 0" rpy="0 ${M_PI/2} 0"/>
+        <!-- <origin xyz="0 0 0" rpy="0 ${M_PI/2} 0"/> -->
         <update_rate>30</update_rate>
         <camera>
@@ -74,5 +74,5 @@
       <enable_wind>0</enable_wind>
       <kinematic>0</kinematic>
-      <gravity>1</gravity>
+      <!-- <gravity>1</gravity> -->
       <!--<mu>1</mu>-->
       <mu2>1</mu2>
@@ -85,5 +85,5 @@
       <min_depth>0</min_depth>-->
       <sensor name="${camera_name}fisheye2" type="wideanglecamera">
-        <origin xyz="0 0 0" rpy="0 ${M_PI/2} 0"/>
+        <!-- <origin xyz="0 0 0" rpy="0 ${M_PI/2} 0"/> -->
         <update_rate>30</update_rate>
         <camera>

File: urdf/_t265.urdf.xacro (robot description, xacro)
@@ -56,5 +56,5 @@
     <!-- camera body, with origin at camera_link -->
     <joint name="${name}_link_joint" type="fixed">
-      <origin xyz="0 0 0" rpy="0 0 0"/>
+      <origin xyz="0 0 0" rpy="${M_PI / 2} 0 -${M_PI / 2}"/>
       <parent link="${name}_pose_frame"/>
       <child link="${name}_link"/>

Commit message: added aligned_depth_to_color for d435 and d435i
as described in the offical [IntelRealSense/realsense-ros/README.md](https://github.com/IntelRealSense/realsense-ros/blob/development/README.md) when the param align_depth is set true, the topics /camera/aligned_depth_to_color/image_raw and /camera/aligned_depth_to_color/camera_info.
To lighten the simulation (differently for the real camera) the /camera/depth/image_rect_raw and /camera/depth/camera_info are removed when the align_depth=true.

File: urdf/_d435.gazebo.xacro (robot description, xacro)
@@ -1,6 +1,7 @@
 <?xml version="1.0"?>
 <!--
-Aknolegment: This file was copied from the realsense repository of
+Aknolegment: This file was originally copied from the realsense repository of
 pal-robotics-forks( https://github.com/pal-robotics-forks/realsense/ )
+and then modified.
 License: Apache 2.0. See LICENSE file in root directory.
 Copyright(c) 2017 PAL Robotics, S.L. All Rights Reserved
@@ -8,5 +9,5 @@
 -->
 <robot xmlns:xacro="http://ros.org/wiki/xacro">
-  <xacro:macro name="gazebo_d435" params="camera_name reference_link topics_ns depth_optical_frame color_optical_frame infrared1_optical_frame infrared2_optical_frame" >
+  <xacro:macro name="gazebo_d435" params="camera_name reference_link topics_ns depth_optical_frame color_optical_frame infrared1_optical_frame infrared2_optical_frame enable_pointCloud:=false align_depth:=false">
     <!-- Load parameters to model's main link-->
     <xacro:property name="deg_to_rad" value="0.01745329251994329577"/>
@@ -119,21 +120,29 @@
       	<colorUpdateRate>60.0</colorUpdateRate>
       	<infraredUpdateRate>60.0</infraredUpdateRate>
-      	<depthTopicName>depth/image_raw</depthTopicName>
-      	<depthCameraInfoTopicName>depth/camera_info</depthCameraInfoTopicName>
       	<colorTopicName>color/image_raw</colorTopicName>
       	<colorCameraInfoTopicName>color/camera_info</colorCameraInfoTopicName>
-      	<infrared1TopicName>infra1/image_raw</infrared1TopicName>
+      	<infrared1TopicName>infra1/image_rect_raw</infrared1TopicName>
       	<infrared1CameraInfoTopicName>infra1/camera_info</infrared1CameraInfoTopicName>
-      	<infrared2TopicName>infra2/image_raw</infrared2TopicName>
+      	<infrared2TopicName>infra2/image_rect_raw</infrared2TopicName>
       	<infrared2CameraInfoTopicName>infra2/camera_info</infrared2CameraInfoTopicName>
       	<colorOpticalframeName>${color_optical_frame}</colorOpticalframeName>
-      	<depthOpticalframeName>${depth_optical_frame}</depthOpticalframeName>
       	<infrared1OpticalframeName>${infrared1_optical_frame}</infrared1OpticalframeName>
       	<infrared2OpticalframeName>${infrared2_optical_frame}</infrared2OpticalframeName>
       	<rangeMinDepth>0.2</rangeMinDepth>
       	<rangeMaxDepth>10.0</rangeMaxDepth>
-      	<pointCloud>true</pointCloud>
-      	<pointCloudTopicName>depth/points</pointCloudTopicName>
+      	<pointCloud>${enable_pointCloud}</pointCloud>
+      	<pointCloudTopicName>depth/color/points</pointCloudTopicName>
       	<pointCloudCutoff>0.5</pointCloudCutoff>
+        <!-- align-depth settings -->
+        <xacro:unless value="${align_depth}">
+      	  <depthTopicName>depth/image_rect_raw</depthTopicName>
+      	  <depthCameraInfoTopicName>depth/camera_info</depthCameraInfoTopicName>
+        	<depthOpticalframeName>${depth_optical_frame}</depthOpticalframeName>
+        </xacro:unless>
+        <xacro:if value="${align_depth}">
+      	  <depthTopicName>aligned_depth_to_color/image_raw</depthTopicName>
+      	  <depthCameraInfoTopicName>aligned_depth_to_color/camera_info</depthCameraInfoTopicName>
+      	  <depthOpticalframeName>${color_optical_frame}</depthOpticalframeName>
+        </xacro:if>
       </plugin>
     </gazebo>

File: urdf/_d435.urdf.xacro (robot description, xacro)
@@ -2,5 +2,5 @@
 <!--
 Aknolegment: This file was copied from the realsense repository of
-pal-robotics-forks( https://github.com/pal-robotics-forks/realsense/ )
+pal-robotics-forks( https://github.com/pal-robotics-forks/realsense/ ).
 and then modified.
 License: Apache 2.0. See LICENSE file in root directory.
@@ -12,5 +12,5 @@
   <!--File includes-->
   <xacro:include filename="$(find realsense_gazebo_description)/urdf/_d435.gazebo.xacro"/>
-  <xacro:macro name="sensor_d435" params="name:=camera topics_ns:=camera parent *origin">
+  <xacro:macro name="sensor_d435" params="name:=camera topics_ns:=camera parent enable_pointCloud:=false align_depth:=false *origin">
     <xacro:property name="M_PI" value="3.1415926535897931"/>
     <!-- The following values are approximate, and the camera node
@@ -123,10 +123,12 @@
     <!-- Realsense Gazebo Plugin -->
     <xacro:gazebo_d435  camera_name="${name}"
+                        topics_ns="${topics_ns}"
                         reference_link="${name}_link"
-                        topics_ns="${topics_ns}"
                         depth_optical_frame="${name}_depth_optical_frame"
                         color_optical_frame="${name}_color_optical_frame"
                         infrared1_optical_frame="${name}_left_ir_optical_frame"
                         infrared2_optical_frame="${name}_right_ir_optical_frame"
+                        enable_pointCloud="${enable_pointCloud}"
+                        align_depth="${align_depth}"
     />
   </xacro:macro>

File: urdf/_d435i.gazebo.xacro (robot description, xacro)
@@ -1,5 +1,5 @@
 <?xml version="1.0"?>
 <!--
-Aknolegment: This file was copied from the realsense repository of
+Aknolegment: This file was originally copied from the realsense repository of
 pal-robotics-forks( https://github.com/pal-robotics-forks/realsense/ )
 and then modified.
@@ -9,5 +9,5 @@
 -->
 <robot xmlns:xacro="http://ros.org/wiki/xacro">
-  <xacro:macro name="gazebo_d435i" params="camera_name reference_link topics_ns depth_optical_frame color_optical_frame infrared1_optical_frame infrared2_optical_frame accel_optical_frame gyro_optical_frame enable_pointCloud:=false unite_imu_method:=false">
+  <xacro:macro name="gazebo_d435i" params="camera_name reference_link topics_ns depth_optical_frame color_optical_frame infrared1_optical_frame infrared2_optical_frame accel_optical_frame gyro_optical_frame enable_pointCloud:=false align_depth:=false unite_imu_method:=false">
     <!-- Load parameters to model's main link-->
     <xacro:property name="deg_to_rad" value="0.01745329251994329577"/>
@@ -171,14 +171,11 @@
       	<colorUpdateRate>60.0</colorUpdateRate>
       	<infraredUpdateRate>60.0</infraredUpdateRate>
-      	<depthTopicName>depth/image_raw</depthTopicName>
-      	<depthCameraInfoTopicName>depth/camera_info</depthCameraInfoTopicName>
       	<colorTopicName>color/image_raw</colorTopicName>
       	<colorCameraInfoTopicName>color/camera_info</colorCameraInfoTopicName>
-      	<infrared1TopicName>infra1/image_raw</infrared1TopicName>
+      	<infrared1TopicName>infra1/image_rect_raw</infrared1TopicName>
       	<infrared1CameraInfoTopicName>infra1/camera_info</infrared1CameraInfoTopicName>
-      	<infrared2TopicName>infra2/image_raw</infrared2TopicName>
+      	<infrared2TopicName>infra2/image_rect_raw</infrared2TopicName>
       	<infrared2CameraInfoTopicName>infra2/camera_info</infrared2CameraInfoTopicName>
       	<colorOpticalframeName>${color_optical_frame}</colorOpticalframeName>
-      	<depthOpticalframeName>${depth_optical_frame}</depthOpticalframeName>
       	<infrared1OpticalframeName>${infrared1_optical_frame}</infrared1OpticalframeName>
       	<infrared2OpticalframeName>${infrared2_optical_frame}</infrared2OpticalframeName>
@@ -186,6 +183,17 @@
       	<rangeMaxDepth>10.0</rangeMaxDepth>
       	<pointCloud>${enable_pointCloud}</pointCloud>
-      	<pointCloudTopicName>depth/points</pointCloudTopicName>
+      	<pointCloudTopicName>depth/color/points</pointCloudTopicName>
       	<pointCloudCutoff>0.5</pointCloudCutoff>
+        <!-- align-depth settings -->
+        <xacro:unless value="${align_depth}">
+      	  <depthTopicName>depth/image_rect_raw</depthTopicName>
+      	  <depthCameraInfoTopicName>depth/camera_info</depthCameraInfoTopicName>
+        	<depthOpticalframeName>${depth_optical_frame}</depthOpticalframeName>
+        </xacro:unless>
+        <xacro:if value="${align_depth}">
+      	  <depthTopicName>aligned_depth_to_color/image_raw</depthTopicName>
+      	  <depthCameraInfoTopicName>aligned_depth_to_color/camera_info</depthCameraInfoTopicName>
+      	  <depthOpticalframeName>${color_optical_frame}</depthOpticalframeName>
+        </xacro:if>
       </plugin>
     </gazebo>

File: urdf/_d435i.urdf.xacro (robot description, xacro)
@@ -12,5 +12,5 @@
   <!--File includes-->
   <xacro:include filename="$(find realsense_gazebo_description)/urdf/_d435i.gazebo.xacro"/>
-  <xacro:macro name="sensor_d435i" params="name:=camera topics_ns:=camera parent enable_pointCloud:=false unite_imu_method:=false *origin">
+  <xacro:macro name="sensor_d435i" params="name:=camera topics_ns:=camera parent enable_pointCloud:=false align_depth:=false unite_imu_method:=false *origin">
     <xacro:property name="M_PI" value="3.1415926535897931"/>
     <!-- The following values are approximate, and the camera node
@@ -149,6 +149,6 @@
     <!-- Realsense Gazebo Plugin -->
     <xacro:gazebo_d435i camera_name="${name}"
+                        topics_ns="${topics_ns}"
                         reference_link="${name}_link"
-                        topics_ns="${topics_ns}"
                         depth_optical_frame="${name}_depth_optical_frame"
                         color_optical_frame="${name}_color_optical_frame"
@@ -159,4 +159,5 @@
                         enable_pointCloud="${enable_pointCloud}"
                         unite_imu_method="${unite_imu_method}"
+                        align_depth="${align_depth}"
     />
   </xacro:macro>

File: urdf/multicamera.urdf.xacro (robot description, xacro)
@@ -4,5 +4,6 @@
   <!-- d435  frame definition can be found at https://github.com/IntelRealSense/librealsense/blob/master/doc/d435i.md -->
   <xacro:include filename="$(find realsense_gazebo_description)/urdf/_d435.urdf.xacro"/>
-  <xacro:sensor_d435 parent="base_link" name="D435_camera" topics_ns="D435_camera">
+  <xacro:sensor_d435  parent="base_link" name="D435_camera" topics_ns="D435_camera"
+                      enable_pointCloud="true" align_depth="true">
     <origin xyz="0.0 -0.5 0.1" rpy="0.0 0.0 0.0"/>
   </xacro:sensor_d435>
@@ -10,5 +11,6 @@
   <xacro:include filename="$(find realsense_gazebo_description)/urdf/_d435i.urdf.xacro"/>
   <xacro:sensor_d435i parent="base_link" name="D435i_camera" topics_ns="D435i_camera"
-                      enable_pointCloud="true" unite_imu_method="copy"> <!-- unite_imu_method can be false, copy or linear_interpolation -->
+                      enable_pointCloud="true" align_depth="true"
+                      unite_imu_method="copy"> <!-- unite_imu_method can be false, copy or linear_interpolation -->
     <origin xyz="0.0 0.5 0.1" rpy="0.0 0.0 0.0"/>
   </xacro:sensor_d435i>
