Commit message: allow changes of camera resolution and framerate

File: urdf/_d435.gazebo.xacro (robot description, xacro)
@@ -9,5 +9,23 @@
 -->
 <robot xmlns:xacro="http://ros.org/wiki/xacro">
-  <xacro:macro name="gazebo_d435" params="camera_name reference_link topics_ns depth_optical_frame color_optical_frame infrared1_optical_frame infrared2_optical_frame enable_pointCloud:=false align_depth:=false">
+  <xacro:macro name="gazebo_d435" params="reference_link
+                                          camera_name:=camera
+                                          topics_ns:=camera
+                                          depth_optical_frame
+                                          color_optical_frame
+                                          infrared1_optical_frame
+                                          infrared2_optical_frame
+                                          depth_width:=1280
+                                          depth_height:=720
+                                          depth_fps:=30
+                                          color_width:=1920
+                                          color_height:=1080
+                                          color_fps:=30
+                                          infra_width:=640
+                                          infra_height:=480
+                                          infra_fps:=30
+                                          align_depth:=false
+                                          enable_pointCloud:=false
+                                          ">
     <!-- Load parameters to model's main link-->
     <xacro:property name="deg_to_rad" value="0.01745329251994329577"/>
@@ -30,6 +48,6 @@
           <horizontal_fov>${69.4*deg_to_rad}</horizontal_fov>
           <image>
-            <width>1920</width>
-            <height>1080</height>
+            <width>${color_width}</width>
+            <height>${color_height}</height>
             <format>RGB_INT8</format>
           </image>
@@ -45,5 +63,5 @@
         </camera>
         <always_on>1</always_on>
-        <update_rate>30</update_rate>
+        <update_rate>${color_fps}</update_rate>
         <visualize>1</visualize>
       </sensor>
@@ -52,6 +70,6 @@
           <horizontal_fov>${85.2*deg_to_rad}</horizontal_fov>
           <image>
-            <width>1280</width>
-            <height>720</height>
+            <width>${infra_width}</width>
+            <height>${infra_height}</height>
             <format>L_INT8</format>
           </image>
@@ -67,5 +85,5 @@
         </camera>
         <always_on>1</always_on>
-        <update_rate>90</update_rate>
+        <update_rate>${infra_fps}</update_rate>
         <visualize>0</visualize>
       </sensor>
@@ -74,6 +92,6 @@
           <horizontal_fov>${85.2*deg_to_rad}</horizontal_fov>
           <image>
-            <width>1280</width>
-            <height>720</height>
+            <width>${infra_width}</width>
+            <height>${infra_height}</height>
             <format>L_INT8</format>
           </image>
@@ -89,5 +107,5 @@
         </camera>
         <always_on>1</always_on>
-        <update_rate>90</update_rate>
+        <update_rate>${infra_fps}</update_rate>
         <visualize>0</visualize>
       </sensor>
@@ -96,6 +114,6 @@
           <horizontal_fov>${85.2*deg_to_rad}</horizontal_fov>
           <image>
-            <width>1280</width>
-            <height>720</height>
+            <width>${depth_width}</width>
+            <height>${depth_height}</height>
           </image>
           <clip>
@@ -110,5 +128,5 @@
         </camera>
         <always_on>1</always_on>
-        <update_rate>90</update_rate>
+        <update_rate>${depth_fps}</update_rate>
         <visualize>0</visualize>
       </sensor>
@@ -117,7 +135,7 @@
       <plugin name="${topics_ns}" filename="librealsense_gazebo_plugin.so">
         <prefix>${camera_name}</prefix>
-      	<depthUpdateRate>60.0</depthUpdateRate>
-      	<colorUpdateRate>60.0</colorUpdateRate>
-      	<infraredUpdateRate>60.0</infraredUpdateRate>
+      	<depthUpdateRate>${depth_fps}</depthUpdateRate>
+      	<colorUpdateRate>${color_fps}</colorUpdateRate>
+      	<infraredUpdateRate>${infra_fps}</infraredUpdateRate>
       	<colorTopicName>color/image_raw</colorTopicName>
       	<colorCameraInfoTopicName>color/camera_info</colorCameraInfoTopicName>

File: urdf/_d435.urdf.xacro (robot description, xacro)
@@ -12,5 +12,19 @@
   <!--File includes-->
   <xacro:include filename="$(find realsense_gazebo_description)/urdf/_d435.gazebo.xacro"/>
-  <xacro:macro name="sensor_d435" params="name:=camera topics_ns:=camera parent enable_pointCloud:=false align_depth:=false *origin">
+  <xacro:macro name="sensor_d435" params="parent
+                                          name:=camera
+                                          topics_ns:=camera
+                                          align_depth:=false
+                                          enable_pointCloud:=false
+                                          depth_width:=1280
+                                          depth_height:=720
+                                          depth_fps:=30
+                                          infra_width:=640
+                                          infra_height:=480
+                                          infra_fps:=30
+                                          color_width:=1920
+                                          color_height:=1080
+                                          color_fps:=30
+                                          *origin">
     <xacro:property name="M_PI" value="3.1415926535897931"/>
     <!-- The following values are approximate, and the camera node
@@ -126,9 +140,18 @@
                         reference_link="${name}_link"
                         depth_optical_frame="${name}_depth_optical_frame"
+                        depth_width="${depth_width}"
+                        depth_height="${depth_height}"
+                        depth_fps="${depth_fps}"
                         color_optical_frame="${name}_color_optical_frame"
+                        color_width="${color_width}"
+                        color_height="${color_height}"
+                        color_fps="${color_fps}"
                         infrared1_optical_frame="${name}_left_ir_optical_frame"
                         infrared2_optical_frame="${name}_right_ir_optical_frame"
+                        infra_width="${infra_width}"
+                        infra_height="${infra_height}"
+                        infra_fps="${infra_fps}"
+                        align_depth="${align_depth}"
                         enable_pointCloud="${enable_pointCloud}"
-                        align_depth="${align_depth}"
     />
   </xacro:macro>

File: urdf/_d435i.gazebo.xacro (robot description, xacro)
@@ -9,5 +9,28 @@
 -->
 <robot xmlns:xacro="http://ros.org/wiki/xacro">
-  <xacro:macro name="gazebo_d435i" params="camera_name reference_link topics_ns depth_optical_frame color_optical_frame infrared1_optical_frame infrared2_optical_frame accel_optical_frame gyro_optical_frame enable_pointCloud:=false align_depth:=false unite_imu_method:=false">
+  <xacro:macro name="gazebo_d435i" params=" reference_link
+                                            camera_name:=camera
+                                            topics_ns:=camera
+                                            depth_optical_frame
+                                            color_optical_frame
+                                            infrared1_optical_frame
+                                            infrared2_optical_frame
+                                            accel_optical_frame
+                                            gyro_optical_frame
+                                            align_depth:=false
+                                            enable_pointCloud:=false
+                                            unite_imu_method:=false
+                                            accel_fps:=250
+                                            gyro_fps:=400
+                                            depth_width:=1280
+                                            depth_height:=720
+                                            depth_fps:=30
+                                            infra_width:=640
+                                            infra_height:=480
+                                            infra_fps:=30
+                                            color_width:=1920
+                                            color_height:=1080
+                                            color_fps:=30
+                                            ">
     <!-- Load parameters to model's main link-->
     <xacro:property name="deg_to_rad" value="0.01745329251994329577"/>
@@ -30,6 +53,6 @@
           <horizontal_fov>${69.4*deg_to_rad}</horizontal_fov>
           <image>
-            <width>1920</width>
-            <height>1080</height>
+            <width>${color_width}</width>
+            <height>${color_height}</height>
             <format>RGB_INT8</format>
           </image>
@@ -45,5 +68,5 @@
         </camera>
         <always_on>1</always_on>
-        <update_rate>30</update_rate>
+        <update_rate>${color_fps}</update_rate>
         <visualize>1</visualize>
       </sensor>
@@ -52,6 +75,6 @@
           <horizontal_fov>${85.2*deg_to_rad}</horizontal_fov>
           <image>
-            <width>1280</width>
-            <height>720</height>
+            <width>${infra_width}</width>
+            <height>${infra_height}</height>
             <format>L_INT8</format>
           </image>
@@ -67,5 +90,5 @@
         </camera>
         <always_on>1</always_on>
-        <update_rate>90</update_rate>
+        <update_rate>${infra_fps}</update_rate>
         <visualize>0</visualize>
       </sensor>
@@ -74,6 +97,6 @@
           <horizontal_fov>${85.2*deg_to_rad}</horizontal_fov>
           <image>
-            <width>1280</width>
-            <height>720</height>
+            <width>${infra_width}</width>
+            <height>${infra_height}</height>
             <format>L_INT8</format>
           </image>
@@ -89,5 +112,5 @@
         </camera>
         <always_on>1</always_on>
-        <update_rate>90</update_rate>
+        <update_rate>${infra_fps}</update_rate>
         <visualize>0</visualize>
       </sensor>
@@ -96,6 +119,6 @@
           <horizontal_fov>${85.2*deg_to_rad}</horizontal_fov>
           <image>
-            <width>1280</width>
-            <height>720</height>
+            <width>${depth_width}</width>
+            <height>${depth_height}</height>
           </image>
           <clip>
@@ -110,5 +133,5 @@
         </camera>
         <always_on>1</always_on>
-        <update_rate>90</update_rate>
+        <update_rate>${depth_fps}</update_rate>
         <visualize>0</visualize>
       </sensor>
@@ -117,5 +140,5 @@
         <sensor name="${camera_name}_imu" type="imu">
           <always_on>true</always_on>
-          <update_rate>300</update_rate>
+          <update_rate>${gyro_fps}</update_rate>
           <topic>${camera_name}/imu/sample</topic>
           <plugin name="{camera_name}imu" filename="libgazebo_ros_imu_sensor.so">
@@ -123,5 +146,5 @@
             <bodyName>${camera_name}_link</bodyName>
             <frameName>${gyro_optical_frame}</frameName>
-            <updateRateHZ>300</updateRateHZ>
+            <updateRateHZ>${gyro_fps}</updateRateHZ>
             <gaussianNoise>0.1</gaussianNoise>
             <xyzOffset>0 0 0</xyzOffset>
@@ -134,10 +157,10 @@
         <sensor name="{camera_name}accel" type="imu">
           <always_on>true</always_on>
-          <update_rate>300</update_rate>
+          <update_rate>${accel_fps}</update_rate>
           <topic>${camera_name}/accel/sample</topic>
           <plugin name="${topics_ns}_accel_plugin" filename="librealsense_gazebo_accel_sensor.so">
             <topicName>${camera_name}/accel/sample</topicName>
             <bodyName>${camera_name}_link</bodyName>
-            <updateRateHZ>300.0</updateRateHZ>
+            <updateRateHZ>${accel_fps}</updateRateHZ>
             <gaussianNoise>0.1</gaussianNoise>
             <xyzOffset>0 0 0</xyzOffset>
@@ -150,10 +173,10 @@
         <sensor name="{camera_name}gyro" type="imu">
           <always_on>true</always_on>
-          <update_rate>300</update_rate>
+          <update_rate>${gyro_fps}</update_rate>
           <topic>${camera_name}/gyro/sample</topic>
           <plugin name="${topics_ns}_gyro_plugin" filename="librealsense_gazebo_gyro_sensor.so">
             <topicName>${camera_name}/gyro/sample</topicName>
             <bodyName>${camera_name}_link</bodyName>
-            <updateRateHZ>300.0</updateRateHZ>
+            <updateRateHZ>${gyro_fps}</updateRateHZ>
             <gaussianNoise>0.1</gaussianNoise>
             <xyzOffset>0 0 0</xyzOffset>
@@ -168,7 +191,7 @@
       <plugin name="${topics_ns}" filename="librealsense_gazebo_plugin.so">
         <prefix>${camera_name}</prefix>
-      	<depthUpdateRate>60.0</depthUpdateRate>
-      	<colorUpdateRate>60.0</colorUpdateRate>
-      	<infraredUpdateRate>60.0</infraredUpdateRate>
+      	<depthUpdateRate>${depth_fps}</depthUpdateRate>
+      	<colorUpdateRate>${color_fps}</colorUpdateRate>
+      	<infraredUpdateRate>${infra_fps}</infraredUpdateRate>
       	<colorTopicName>color/image_raw</colorTopicName>
       	<colorCameraInfoTopicName>color/camera_info</colorCameraInfoTopicName>

File: urdf/_d435i.urdf.xacro (robot description, xacro)
@@ -12,5 +12,22 @@
   <!--File includes-->
   <xacro:include filename="$(find realsense_gazebo_description)/urdf/_d435i.gazebo.xacro"/>
-  <xacro:macro name="sensor_d435i" params="name:=camera topics_ns:=camera parent enable_pointCloud:=false align_depth:=false unite_imu_method:=false *origin">
+  <xacro:macro name="sensor_d435i" params="parent
+                                          name:=camera
+                                          topics_ns:=camera
+                                          align_depth:=false
+                                          enable_pointCloud:=true
+                                          unite_imu_method:=false
+                                          accel_fps:=250
+                                          gyro_fps:=400
+                                          depth_width:=1280
+                                          depth_height:=720
+                                          depth_fps:=30
+                                          infra_width:=640
+                                          infra_height:=480
+                                          infra_fps:=30
+                                          color_width:=1920
+                                          color_height:=1080
+                                          color_fps:=30
+                                          *origin">
     <xacro:property name="M_PI" value="3.1415926535897931"/>
     <!-- The following values are approximate, and the camera node

File: urdf/_t265.gazebo.xacro (robot description, xacro)
@@ -9,5 +9,22 @@
 -->
 <robot xmlns:xacro="http://ros.org/wiki/xacro">
-  <xacro:macro name="gazebo_t265" params="camera_name fisheye1_reference_link fisheye2_reference_link topics_ns fisheye1_optical_frame fisheye2_optical_frame accel_optical_frame gyro_optical_frame pose_frame xyz rpy odom_rate:=200 unite_imu_method:=false">
+  <xacro:macro name="gazebo_t265" params="camera_name topics_ns
+                                          fisheye1_reference_link
+                                          fisheye2_reference_link
+                                          fisheye1_optical_frame
+                                          fisheye2_optical_frame
+                                          fisheye_width:=848
+                                          fisheye_height:=800
+                                          fisheye_fps:=30
+                                          accel_optical_frame
+                                          gyro_optical_frame
+                                          unite_imu_method:=false
+                                          accel_fps:=62.5
+                                          gyro_fps:=200
+                                          pose_frame
+                                          odom_xyz
+                                          odom_rpy
+                                          odom_fps:=200
+                                          ">
     <!-- Load parameters to model's main link-->
     <gazebo reference="${fisheye1_reference_link}">
@@ -27,10 +44,10 @@
       <sensor name="${camera_name}fisheye1" type="wideanglecamera">
         <!-- <origin xyz="0 0 0" rpy="0 ${M_PI/2} 0"/> -->
-        <update_rate>30</update_rate>
+        <update_rate>${fisheye_fps}</update_rate>
         <camera>
           <horizontal_fov>1.95</horizontal_fov>
           <image>
-            <width>848</width>
-            <height>800</height>
+            <width>${fisheye_width}</width>
+            <height>${fisheye_height}</height>
           </image>
           <clip>
@@ -53,5 +70,5 @@
         <plugin name="${camera_name}fisheye1" filename="libgazebo_ros_camera.so">
           <alwaysOn>true</alwaysOn>
-          <updateRate>30.0</updateRate>
+          <updateRate>${fisheye_fps}</updateRate>
           <cameraName>${topics_ns}/fisheye1</cameraName>
           <imageTopicName>image_raw</imageTopicName>
@@ -86,10 +103,10 @@
       <sensor name="${camera_name}fisheye2" type="wideanglecamera">
         <!-- <origin xyz="0 0 0" rpy="0 ${M_PI/2} 0"/> -->
-        <update_rate>30</update_rate>
+        <update_rate>${fisheye_fps}</update_rate>
         <camera>
           <horizontal_fov>2.84</horizontal_fov>
           <image>
-            <width>848</width>
-            <height>800</height>
+            <width>${fisheye_width}</width>
+            <height>${fisheye_height}</height>
           </image>
           <clip>
@@ -113,5 +130,5 @@
         <plugin name="${camera_name}fisheye2" filename="libgazebo_ros_camera.so">
           <alwaysOn>true</alwaysOn>
-          <updateRate>30.0</updateRate>
+          <updateRate>${fisheye_fps}</updateRate>
           <cameraName>${topics_ns}/fisheye2</cameraName>
           <imageTopicName>image_raw</imageTopicName>
@@ -130,5 +147,5 @@
         <sensor name="${camera_name}_imu" type="imu">
           <always_on>true</always_on>
-          <update_rate>300</update_rate>
+          <update_rate>${gyro_fps}</update_rate>
           <topic>${camera_name}/imu/sample</topic>
           <plugin name="{camera_name}imu" filename="libgazebo_ros_imu_sensor.so">
@@ -136,5 +153,5 @@
             <bodyName>${camera_name}_pose_frame</bodyName>
             <frameName>${gyro_optical_frame}</frameName>
-            <updateRateHZ>300</updateRateHZ>
+            <updateRateHZ>${gyro_fps}</updateRateHZ>
             <gaussianNoise>0.1</gaussianNoise>
             <xyzOffset>0 0 0</xyzOffset>
@@ -147,9 +164,9 @@
         <sensor name="{camera_name}accel" type="imu">
           <always_on>true</always_on>
-          <update_rate>300</update_rate>
+          <update_rate>${accel_fps}</update_rate>
           <plugin name="${topics_ns}_accel_plugin" filename="librealsense_gazebo_accel_sensor.so">
             <topicName>${camera_name}/accel/sample</topicName>
             <bodyName>${camera_name}_pose_frame</bodyName>
-            <updateRateHZ>300.0</updateRateHZ>
+            <updateRateHZ>${accel_fps}</updateRateHZ>
             <gaussianNoise>0.1</gaussianNoise>
             <xyzOffset>0 0 0</xyzOffset>
@@ -162,10 +179,10 @@
         <sensor name="{camera_name}gyro" type="imu">
           <always_on>true</always_on>
-          <update_rate>300</update_rate>
+          <update_rate>${gyro_fps}</update_rate>
           <topic>${topics_ns}/gyro/sample</topic>
           <plugin name="${topics_ns}_gyro_plugin" filename="librealsense_gazebo_gyro_sensor.so">
             <topicName>${camera_name}/gyro/sample</topicName>
             <bodyName>${camera_name}_pose_frame</bodyName>
-            <updateRateHZ>300.0</updateRateHZ>
+            <updateRateHZ>${gyro_fps}</updateRateHZ>
             <gaussianNoise>0.1</gaussianNoise>
             <xyzOffset>0 0 0</xyzOffset>
@@ -181,11 +198,11 @@
       <plugin name="p3d_base_controller" filename="libgazebo_ros_p3d.so">
             <alwaysOn>true</alwaysOn>
-            <updateRate>${odom_rate}</updateRate>
+            <updateRate>${odom_fps}</updateRate>
             <bodyName>${pose_frame}</bodyName>
             <topicName>${topics_ns}/odom/sample</topicName>
             <gaussianNoise>0.01</gaussianNoise>
             <frameName>world</frameName>
-            <xyzOffsets>${xyz}</xyzOffsets>
-            <rpyOffsets>${rpy}</rpyOffsets>
+            <xyzOffsets>${odom_xyz}</xyzOffsets>
+            <rpyOffsets>${odom_rpy}</rpyOffsets>
         </plugin>
     </gazebo>
