Commit message: allow changes of camera resolution and framerate

File: urdf/_t265.urdf.xacro (robot description, xacro)
@@ -3,16 +3,29 @@
 Aknolegment: This file was copied from the realsense repository of
 pal-robotics-forks( https://github.com/pal-robotics-forks/realsense/ ).
-Lines 17,47,54 were then modified.
+and then modified.
 License: Apache 2.0. See LICENSE file in root directory.
 Copyright(c) 2017 Intel Corporation. All Rights Reserved
 This is the URDF model for the Intel RealSense T265 camera, in it's
 aluminum peripherial evaluation case.
+The camera specs can be found at https://www.intelrealsense.com/how-to-getting-imu-data-from-d435i-and-t265/ .
 -->
 <robot name="sensor_t265" xmlns:xacro="http://ros.org/wiki/xacro">
   <!--File includes-->
   <xacro:include filename="$(find realsense_gazebo_description)/urdf/_t265.gazebo.xacro"/>
-  <!-- tx,ty,tz,rr,rp,ry (xyz rpy) are the transformation from the robot base_link to the camera reference frame (camerea_pose_frame)
+    <!-- odom_xyz, odom_rpy params are the transformation from the robot base_link to the camera reference frame (camerea_pose_frame)
   they are needed for the simulation of the camera slam capabilities -->
-  <xacro:macro name="sensor_t265" params="parent xyz rpy name:=camera topics_ns:=camera odom_rate:=200 unite_imu_method:=false *origin">
+  <xacro:macro name="sensor_t265" params="parent
+                                          name:=camera
+                                          topics_ns:=camera
+                                          unite_imu_method:=false
+                                          accel_fps:=62.5
+                                          gyro_fps:=200
+                                          fisheye_width:=848
+                                          fisheye_height:=800
+                                          fisheye_fps:=30
+                                          odom_xyz
+                                          odom_rpy
+                                          odom_fps:=262
+                                          *origin">
     <xacro:property name="M_PI" value="3.1415926535897931"/>
     <!-- The following values are approximate, and the camera node
@@ -111,23 +124,22 @@
     <link name="${name}_gyro_optical_frame"/>
     <!-- Realsense Gazebo Plugin -->
-    <xacro:gazebo_t265  camera_name="${name}"
-                        topics_ns="${topics_ns}"
-                        pose_frame="${name}_pose_frame"
+    <xacro:gazebo_t265  camera_name="${name}" topics_ns="${topics_ns}"
                         fisheye1_reference_link="${name}_fisheye1_rgb_frame"
                         fisheye2_reference_link="${name}_fisheye2_rgb_frame"
                         fisheye1_optical_frame="${name}_fisheye1_optical_frame"
                         fisheye2_optical_frame="${name}_fisheye2_optical_frame"
+                        fisheye_width="${fisheye_width}"
+                        fisheye_height="${fisheye_height}"
+                        fisheye_fps="${fisheye_fps}"
                         accel_optical_frame="${name}_accel_optical_frame"
                         gyro_optical_frame="${name}_gyro_optical_frame"
-                        odom_rate="${odom_rate}"
-                        xyz="${xyz}"
-                        rpy="${rpy}"
                         unite_imu_method="${unite_imu_method}"
+                        accel_fps="${accel_fps}"
+                        gyro_fps="${gyro_fps}"
+                        pose_frame="${name}_pose_frame"
+                        odom_xyz="${odom_xyz}"
+                        odom_rpy="${odom_rpy}"
+                        odom_fps="${odom_fps}"
     />
-    <!--
-                        xyz="${tx} ${ty} ${tz}"
-                        rpy="${rr + M_PI} ${rp} ${ry + M_PI}"
-    />
-    -->
   </xacro:macro>
 </robot>

File: urdf/multicamera.urdf.xacro (robot description, xacro)
@@ -4,13 +4,10 @@
   <!-- d435  frame definition can be found at https://github.com/IntelRealSense/librealsense/blob/master/doc/d435i.md -->
   <xacro:include filename="$(find realsense_gazebo_description)/urdf/_d435.urdf.xacro"/>
-  <xacro:sensor_d435  parent="base_link" name="D435_camera" topics_ns="D435_camera"
-                      enable_pointCloud="true" align_depth="true">
+  <xacro:sensor_d435  parent="base_link" name="D435_camera" topics_ns="D435_camera" >
     <origin xyz="0.0 -0.5 0.1" rpy="0.0 0.0 0.0"/>
   </xacro:sensor_d435>
   <!-- d435i frame definition can be found at https://github.com/IntelRealSense/librealsense/blob/master/doc/d435i.md -->
   <xacro:include filename="$(find realsense_gazebo_description)/urdf/_d435i.urdf.xacro"/>
-  <xacro:sensor_d435i parent="base_link" name="D435i_camera" topics_ns="D435i_camera"
-                      enable_pointCloud="true" align_depth="true"
-                      unite_imu_method="copy"> <!-- unite_imu_method can be false, copy or linear_interpolation -->
+  <xacro:sensor_d435i parent="base_link" name="D435i_camera" topics_ns="D435i_camera">
     <origin xyz="0.0 0.5 0.1" rpy="0.0 0.0 0.0"/>
   </xacro:sensor_d435i>
@@ -18,6 +15,5 @@
   <xacro:include filename="$(find realsense_gazebo_description)/urdf/_t265.urdf.xacro"/>
   <xacro:sensor_t265  parent="base_link" name="T265_camera" topics_ns="T265_camera"
-                      xyz="0.0 0.0 0.25" rpy="0.0 0.0 0.0"
-                      unite_imu_method="false"> <!-- unite_imu_method can be false, copy or linear_interpolation -->
+                      odom_xyz="0.0 0.0 0.25" odom_rpy="0.0 0.0 0.0">
     <origin xyz="0.0 0.0 0.25" rpy="0.0 0.0 0.0"/>
   </xacro:sensor_t265>

Commit message: allow to disable <visualize>

File: urdf/_d435.gazebo.xacro (robot description, xacro)
@@ -27,4 +27,5 @@
                                           align_depth:=false
                                           enable_pointCloud:=false
+                                          visualize:=false
                                           ">
     <!-- Load parameters to model's main link-->
@@ -64,5 +65,5 @@
         <always_on>1</always_on>
         <update_rate>${color_fps}</update_rate>
-        <visualize>1</visualize>
+        <visualize>${visualize}</visualize>
       </sensor>
       <sensor name="${camera_name}ired1" type="camera">
@@ -86,5 +87,5 @@
         <always_on>1</always_on>
         <update_rate>${infra_fps}</update_rate>
-        <visualize>0</visualize>
+        <visualize>false</visualize>
       </sensor>
       <sensor name="${camera_name}ired2" type="camera">
@@ -108,5 +109,5 @@
         <always_on>1</always_on>
         <update_rate>${infra_fps}</update_rate>
-        <visualize>0</visualize>
+        <visualize>false</visualize>
       </sensor>
       <sensor name="${camera_name}depth" type="depth">
@@ -129,5 +130,5 @@
         <always_on>1</always_on>
         <update_rate>${depth_fps}</update_rate>
-        <visualize>0</visualize>
+        <visualize>false</visualize>
       </sensor>
     </gazebo>

File: urdf/_d435.urdf.xacro (robot description, xacro)
@@ -26,4 +26,5 @@
                                           color_height:=1080
                                           color_fps:=30
+                                          visualize:=false
                                           *origin">
     <xacro:property name="M_PI" value="3.1415926535897931"/>
@@ -152,6 +153,7 @@
                         infra_height="${infra_height}"
                         infra_fps="${infra_fps}"
+                        enable_pointCloud="${enable_pointCloud}"
                         align_depth="${align_depth}"
-                        enable_pointCloud="${enable_pointCloud}"
+                        visualize="${visualize}"
     />
   </xacro:macro>

File: urdf/_d435i.gazebo.xacro (robot description, xacro)
@@ -18,4 +18,5 @@
                                             accel_optical_frame
                                             gyro_optical_frame
+                                            visualize:=false
                                             align_depth:=false
                                             enable_pointCloud:=false
@@ -69,5 +70,5 @@
         <always_on>1</always_on>
         <update_rate>${color_fps}</update_rate>
-        <visualize>1</visualize>
+        <visualize>${visualize}</visualize>
       </sensor>
       <sensor name="${camera_name}ired1" type="camera">
@@ -91,5 +92,5 @@
         <always_on>1</always_on>
         <update_rate>${infra_fps}</update_rate>
-        <visualize>0</visualize>
+        <visualize>false</visualize>
       </sensor>
       <sensor name="${camera_name}ired2" type="camera">
@@ -113,5 +114,5 @@
         <always_on>1</always_on>
         <update_rate>${infra_fps}</update_rate>
-        <visualize>0</visualize>
+        <visualize>false</visualize>
       </sensor>
       <sensor name="${camera_name}depth" type="depth">
@@ -134,5 +135,5 @@
         <always_on>1</always_on>
         <update_rate>${depth_fps}</update_rate>
-        <visualize>0</visualize>
+        <visualize>false</visualize>
       </sensor>
       <!-- IMU -->

File: urdf/_d435i.urdf.xacro (robot description, xacro)
@@ -15,4 +15,5 @@
                                           name:=camera
                                           topics_ns:=camera
+                                          visualize:=false
                                           align_depth:=false
                                           enable_pointCloud:=true
@@ -177,4 +178,5 @@
                         unite_imu_method="${unite_imu_method}"
                         align_depth="${align_depth}"
+                        visualize="${visualize}"
     />
   </xacro:macro>

File: urdf/multicamera.urdf.xacro (robot description, xacro)
@@ -4,11 +4,11 @@
   <!-- d435  frame definition can be found at https://github.com/IntelRealSense/librealsense/blob/master/doc/d435i.md -->
   <xacro:include filename="$(find realsense_gazebo_description)/urdf/_d435.urdf.xacro"/>
-  <xacro:sensor_d435  parent="base_link" name="D435_camera" topics_ns="D435_camera" >
-    <origin xyz="0.0 -0.5 0.1" rpy="0.0 0.0 0.0"/>
+  <xacro:sensor_d435  parent="base_link" name="D435_camera" topics_ns="D435_camera" visualize="true">
+    <origin xyz="0.0 -0.5 0" rpy="0.0 0.0 0.0"/>
   </xacro:sensor_d435>
   <!-- d435i frame definition can be found at https://github.com/IntelRealSense/librealsense/blob/master/doc/d435i.md -->
   <xacro:include filename="$(find realsense_gazebo_description)/urdf/_d435i.urdf.xacro"/>
   <xacro:sensor_d435i parent="base_link" name="D435i_camera" topics_ns="D435i_camera">
-    <origin xyz="0.0 0.5 0.1" rpy="0.0 0.0 0.0"/>
+    <origin xyz="0.0 0.5 0" rpy="0.0 0.0 0.0"/>
   </xacro:sensor_d435i>
   <!-- t265  frame definition can be found at https://github.com/IntelRealSense/librealsense/blob/master/doc/t265.md -->
@@ -16,5 +16,18 @@
   <xacro:sensor_t265  parent="base_link" name="T265_camera" topics_ns="T265_camera"
                       odom_xyz="0.0 0.0 0.25" odom_rpy="0.0 0.0 0.0">
-    <origin xyz="0.0 0.0 0.25" rpy="0.0 0.0 0.0"/>
+    <origin xyz="0.0 0.0 0.15" rpy="0.0 0.0 0.0"/>
   </xacro:sensor_t265>
+  <!-- add a cone, just to have something to see -->
+  <joint name="cone_joint" type="fixed">
+          <parent link="base_link"/>
+          <child link="cone_link"/>
+          <origin xyz="4 0 0" rpy="0 0 0"/>
+  </joint>
+  <link name='cone_link'>
+    <visual>
+      <geometry>
+        <mesh filename="model://construction_cone/meshes/construction_cone.dae" scale="10 10 10"/>
+      </geometry>
+    </visual>
+  </link>
 </robot>

File: urdf/multicamera_params.urdf.xacro (robot description, xacro)
@@ -7,4 +7,5 @@
                       enable_pointCloud="false"
                       align_depth="false"
+                      visualize:="false"
                       depth_width="1280"
                       depth_height="720"
@@ -17,5 +18,5 @@
                       color_fps="30"
                       >
-    <origin xyz="0.0 -0.5 0.1" rpy="0.0 0.0 0.0"/>
+    <origin xyz="0.0 -0.5 0.0" rpy="0.0 0.0 0.0"/>
   </xacro:sensor_d435>
   <!-- d435i frame definition can be found at https://github.com/IntelRealSense/librealsense/blob/master/doc/d435i.md -->
@@ -25,4 +26,5 @@
                       enable_pointCloud="true"
                       align_depth="false"
+                      visualize:="false"
                       unite_imu_method="false"
                       accel_fps="250"
@@ -38,5 +40,5 @@
                       color_fps="30"
                       >
-    <origin xyz="0.0 0.5 0.1" rpy="0.0 0.0 0.0"/>
+    <origin xyz="0.0 0.5 0.0" rpy="0.0 0.0 0.0"/>
   </xacro:sensor_d435i>
   <!-- t265  frame definition can be found at https://github.com/IntelRealSense/librealsense/blob/master/doc/t265.md -->
@@ -55,5 +57,18 @@
                       gyro_fps="200"
                       >
-    <origin xyz="0.0 0.0 0.25" rpy="0.0 0.0 0.0"/>
+    <origin xyz="0.0 0.0 0.15" rpy="0.0 0.0 0.0"/>
   </xacro:sensor_t265>
+  <!-- add a cone, just to have something to see -->
+  <joint name="cone_joint" type="fixed">
+          <parent link="base_link"/>
+          <child link="cone_link"/>
+          <origin xyz="4 0 0" rpy="0 0 0"/>
+  </joint>
+  <link name='cone_link'>
+    <visual>
+      <geometry>
+        <mesh filename="model://construction_cone/meshes/construction_cone.dae" scale="10 10 10"/>
+      </geometry>
+    </visual>
+  </link>
 </robot>

Commit message: added clip_distance

File: urdf/_d435.gazebo.xacro (robot description, xacro)
@@ -16,4 +16,5 @@
                                           infrared1_optical_frame
                                           infrared2_optical_frame
+                                          clip_distance:=-1.0
                                           depth_width:=1280
                                           depth_height:=720
@@ -130,5 +131,10 @@
           <clip>
             <near>0.1</near>
-            <far>100</far>
+            <xacro:unless value="${clip_distance > 0.0}">
+              <far>100</far>
+            </xacro:unless>
+            <xacro:if value="${clip_distance > 0.0}">
+              <far>${clip_distance}</far>
+            </xacro:if>
           </clip>
           <noise>
@@ -166,5 +172,10 @@
         <!-- Depth camera settings -->
       	<rangeMinDepth>0.2</rangeMinDepth>
-      	<rangeMaxDepth>10.0</rangeMaxDepth>
+        <xacro:unless value="${clip_distance > 0.0}">
+      	  <rangeMaxDepth>10.0</rangeMaxDepth>
+        </xacro:unless>
+        <xacro:if value="${clip_distance > 0.0}">
+          <rangeMaxDepth>${clip_distance}</rangeMaxDepth>
+        </xacro:if>
         <xacro:unless value="${align_depth}">
         	<depthUpdateRate>${depth_fps}</depthUpdateRate>

File: urdf/_d435.urdf.xacro (robot description, xacro)
@@ -17,4 +17,5 @@
                                           align_depth:=false
                                           enable_pointCloud:=false
+                                          clip_distance:=-1.0
                                           depth_width:=1280
                                           depth_height:=720
@@ -154,4 +155,5 @@
                         infra_fps="${infra_fps}"
                         enable_pointCloud="${enable_pointCloud}"
+                        clip_distance="${clip_distance}"
                         align_depth="${align_depth}"
                         visualize="${visualize}"

File: urdf/_d435i.gazebo.xacro (robot description, xacro)
@@ -24,4 +24,5 @@
                                             accel_fps:=250
                                             gyro_fps:=400
+                                            clip_distance:=-1.0
                                             depth_width:=1280
                                             depth_height:=720
@@ -135,5 +136,10 @@
           <clip>
             <near>0.1</near>
-            <far>100</far>
+            <xacro:unless value="${clip_distance > 0.0}">
+              <far>100</far>
+            </xacro:unless>
+            <xacro:if value="${clip_distance > 0.0}">
+              <far>${clip_distance}</far>
+            </xacro:if>
           </clip>
           <noise>
@@ -222,5 +228,10 @@
         <!-- Depth camera settings -->
       	<rangeMinDepth>0.2</rangeMinDepth>
-      	<rangeMaxDepth>10.0</rangeMaxDepth>
+        <xacro:unless value="${clip_distance > 0.0}">
+      	  <rangeMaxDepth>10.0</rangeMaxDepth>
+        </xacro:unless>
+        <xacro:if value="${clip_distance > 0.0}">
+          <rangeMaxDepth>${clip_distance}</rangeMaxDepth>
+        </xacro:if>
         <xacro:unless value="${align_depth}">
         	<depthUpdateRate>${depth_fps}</depthUpdateRate>

File: urdf/_d435i.urdf.xacro (robot description, xacro)
@@ -21,4 +21,5 @@
                                           accel_fps:=250
                                           gyro_fps:=400
+                                          clip_distance:=-1.0
                                           depth_width:=1280
                                           depth_height:=720
@@ -188,4 +189,5 @@
                         enable_pointCloud="${enable_pointCloud}"
                         unite_imu_method="${unite_imu_method}"
+                        clip_distance="${clip_distance}"
                         align_depth="${align_depth}"
                         visualize="${visualize}"

File: urdf/multicamera.urdf.xacro (robot description, xacro)
@@ -5,12 +5,14 @@
   <xacro:include filename="$(find realsense_gazebo_description)/urdf/_d435.urdf.xacro"/>
   <xacro:sensor_d435  parent="base_link" name="D435_camera" topics_ns="D435_camera" visualize="true">
-    <origin xyz="0.0 -0.5 0" rpy="0.0 0.0 0.0"/>
+    <origin xyz="0.0 -0.5 0.0" rpy="0.0 0.0 0.0"/>
   </xacro:sensor_d435>
   <!-- d435i frame definition can be found at https://github.com/IntelRealSense/librealsense/blob/master/doc/d435i.md -->
   <xacro:include filename="$(find realsense_gazebo_description)/urdf/_d435i.urdf.xacro"/>
   <xacro:sensor_d435i parent="base_link" name="D435i_camera" topics_ns="D435i_camera">
-    <origin xyz="0.0 0.5 0" rpy="0.0 0.0 0.0"/>
+    <origin xyz="0.0 0.5 0.0" rpy="0.0 0.0 0.0"/>
   </xacro:sensor_d435i>
   <!-- t265  frame definition can be found at https://github.com/IntelRealSense/librealsense/blob/master/doc/t265.md -->
+  <!-- odom_xyz and odom_rpy paramenters are used as a base for odometry, they represent the trasformation from the robot
+       base_link. unite_imu_method can be "false", "copy" or "linear_interpolation" -->
   <xacro:include filename="$(find realsense_gazebo_description)/urdf/_t265.urdf.xacro"/>
   <xacro:sensor_t265  parent="base_link" name="T265_camera" topics_ns="T265_camera"

File: urdf/multicamera_params.urdf.xacro (robot description, xacro)
@@ -6,4 +6,5 @@
   <xacro:sensor_d435  parent="base_link" name="D435_camera" topics_ns="D435_camera"
                       enable_pointCloud="false"
+                      clip_distance="-1.0"
                       align_depth="false"
                       visualize="false"
@@ -25,4 +26,5 @@
   <xacro:sensor_d435i parent="base_link" name="D435i_camera" topics_ns="D435i_camera"
                       enable_pointCloud="true"
+                      clip_distance="-1.0"
                       align_depth="false"
                       visualize="false"
